File: kicad/isometric-instrument.sch (KiCad schematic (older format))
At the start: 203 parts, among them J1 RJ45, J2 RJ45, J3 RJ45, SW1 SWITCH_INV, SW10 SWITCH_INV, SW11 SWITCH_INV, SW12 SWITCH_INV, SW13 SWITCH_INV, SW14 SWITCH_INV, SW15 SWITCH_INV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

Commit message: gotovo
Connections:
- net at J1.8, R8.2: now also R1.2, R2.2, R3.2, R4.2, R5.2, R6.2, R7.2
