File: kicad/_autosave-isometric-instrument.kicad_pcb (KiCad board)
At the start: 2 copper layers, 203 parts, among them J1 RJ45, J2 RJ45, J3 RJ45, SW1 SWITCH_INV, SW10 SWITCH_INV, SW11 SWITCH_INV, SW12 SWITCH_INV, SW13 SWITCH_INV, SW14 SWITCH_INV, SW15 SWITCH_INV, SW16 SWITCH_INV, SW17 SWITCH_INV, SW18 SWITCH_INV, SW19 SWITCH_INV, SW2 SWITCH_INV, SW20 SWITCH_INV, SW21 SWITCH_INV, SW22 SWITCH_INV, SW23 SWITCH_INV, SW24 SWITCH_INV, SW25 SWITCH_INV, SW26 SWITCH_INV, SW27 SWITCH_INV, SW28 SWITCH_INV, SW29 SWITCH_INV, SW3 SWITCH_INV, SW30 SWITCH_INV, SW31 SWITCH_INV, SW32 SWITCH_INV, SW33 SWITCH_INV, SW34 SWITCH_INV, SW35 SWITCH_INV, SW36 SWITCH_INV, SW37 SWITCH_INV, SW38 SWITCH_INV, SW39 SWITCH_INV, SW4 SWITCH_INV, SW40 SWITCH_INV, SW41 SWITCH_INV, SW42 SWITCH_INV, SW43 SWITCH_INV, SW44 SWITCH_INV, SW45 SWITCH_INV, SW46 SWITCH_INV, SW47 SWITCH_INV, SW48 SWITCH_INV, SW49 SWITCH_INV, SW5 SWITCH_INV, SW50 SWITCH_INV, SW51 SWITCH_INV, SW52 SWITCH_INV, SW53 SWITCH_INV, SW54 SWITCH_INV, SW55 SWITCH_INV, SW56 SWITCH_INV, SW57 SWITCH_INV, SW58 SWITCH_INV, SW59 SWITCH_INV, SW6 SWITCH_INV, SW60 SWITCH_INV, SW61 SWITCH_INV, SW62 SWITCH_INV, SW63 SWITCH_INV, SW64 SWITCH_INV, SW65 SWITCH_INV, SW66 SWITCH_INV, SW67 SWITCH_INV, SW68 SWITCH_INV, SW69 SWITCH_INV, SW7 SWITCH_INV, SW70 SWITCH_INV, SW71 SWITCH_INV, SW72 SWITCH_INV, SW73 SWITCH_INV, SW74 SWITCH_INV, SW75 SWITCH_INV, SW76 SWITCH_INV, SW77 SWITCH_INV, SW78 SWITCH_INV, SW79 SWITCH_INV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

Commit message: gotovo
Other:
- board outline added: 259 x 308 mm
Changed lines of the file:
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@@
     (links 304)
     (no_connects 152)
-    (area 179.949999 68.32051 425.240235 373.537501)
+    (area 179.949999 64.949999 439.050001 373.537501)
     (thickness 1.6)
-    (drawings 582)
+    (drawings 586)
     (tracks 371)
     (zones 0)
@@
     (visible_elements FFFFFF7F)
     (pcbplotparams
-      (layerselection 0x00130_80000001)
+      (layerselection 0x01000_00000000)
       (usegerberextensions false)
       (excludeedgelayer true)
@@
       (padsonsilk false)
       (subtractmaskfromsilk false)
-      (outputformat 1)
+      (outputformat 3)
       (mirror false)
       (drillshape 0)
@@
       (net 108 "Net-(J1-Pad4)"))
   )
+  (gr_line (start 180 373) (end 180 65) (layer Edge.Cuts) (width 0.1))
+  (gr_line (start 439 373) (end 180 373) (layer Edge.Cuts) (width 0.1))
+  (gr_line (start 439 373) (end 439 65) (layer Edge.Cuts) (width 0.1))
+  (gr_line (start 180 65) (end 439 65) (layer Edge.Cuts) (width 0.1))
   (gr_line (start 400 70.989) (end 415 100.989) (layer Dwgs.User) (width 0.1))
   (gr_line (start 400 100.989) (end 415 70.989) (layer Dwgs.User) (width 0.1))
