File: kicad/isometric-instrument.kicad_pcb (KiCad board)
At the start: 2 copper layers, 203 parts, among them J1 RJ45, J2 RJ45, J3 RJ45, SW1 SWITCH_INV, SW10 SWITCH_INV, SW11 SWITCH_INV, SW12 SWITCH_INV, SW13 SWITCH_INV, SW14 SWITCH_INV, SW15 SWITCH_INV, SW16 SWITCH_INV, SW17 SWITCH_INV, SW18 SWITCH_INV, SW19 SWITCH_INV, SW2 SWITCH_INV, SW20 SWITCH_INV, SW21 SWITCH_INV, SW22 SWITCH_INV, SW23 SWITCH_INV, SW24 SWITCH_INV, SW25 SWITCH_INV, SW26 SWITCH_INV, SW27 SWITCH_INV, SW28 SWITCH_INV, SW29 SWITCH_INV, SW3 SWITCH_INV, SW30 SWITCH_INV, SW31 SWITCH_INV, SW32 SWITCH_INV, SW33 SWITCH_INV, SW34 SWITCH_INV, SW35 SWITCH_INV, SW36 SWITCH_INV, SW37 SWITCH_INV, SW38 SWITCH_INV, SW39 SWITCH_INV, SW4 SWITCH_INV, SW40 SWITCH_INV, SW41 SWITCH_INV, SW42 SWITCH_INV, SW43 SWITCH_INV, SW44 SWITCH_INV, SW45 SWITCH_INV, SW46 SWITCH_INV, SW47 SWITCH_INV, SW48 SWITCH_INV, SW49 SWITCH_INV, SW5 SWITCH_INV, SW50 SWITCH_INV, SW51 SWITCH_INV, SW52 SWITCH_INV, SW53 SWITCH_INV, SW54 SWITCH_INV, SW55 SWITCH_INV, SW56 SWITCH_INV, SW57 SWITCH_INV, SW58 SWITCH_INV, SW59 SWITCH_INV, SW6 SWITCH_INV, SW60 SWITCH_INV, SW61 SWITCH_INV, SW62 SWITCH_INV, SW63 SWITCH_INV, SW64 SWITCH_INV, SW65 SWITCH_INV, SW66 SWITCH_INV, SW67 SWITCH_INV, SW68 SWITCH_INV, SW69 SWITCH_INV, SW7 SWITCH_INV, SW70 SWITCH_INV, SW71 SWITCH_INV, SW72 SWITCH_INV, SW73 SWITCH_INV, SW74 SWITCH_INV, SW75 SWITCH_INV, SW76 SWITCH_INV, SW77 SWITCH_INV, SW78 SWITCH_INV, SW79 SWITCH_INV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

Commit message: gotovo
Parts:
- moved D91 609.9 mm to (409.5, 250.0), turned to 90 degrees
- moved D89 607.0 mm to (409.5, 320.0), turned to 90 degrees
- moved D93 590.3 mm to (409.5, 180.0), turned to 90 degrees
- moved D88 590.1 mm to (389.5, 75.0), turned to 90 degrees
- moved D90 582.4 mm to (409.5, 285.0), turned to 90 degrees
- moved D81 582.3 mm to (389.5, 320.0), turned to 90 degrees
- moved D76 578.3 mm to (369.5, 215.0), turned to 90 degrees
- moved D73 571.2 mm to (369.5, 320.0), turned to 90 degrees
- moved D85 569.9 mm to (389.5, 180.0), turned to 90 degrees
- moved D84 561.3 mm to (389.5, 215.0), turned to 90 degrees
- moved R1 551.4 mm to (419.5, 320.0), turned to 270 degrees
- moved R6 549.1 mm to (419.5, 145.0), turned to 270 degrees
- moved D83 545.9 mm to (389.5, 250.0), turned to 90 degrees
- moved D75 544.9 mm to (369.5, 250.0), turned to 90 degrees
- moved D87 542.8 mm to (389.5, 110.0), turned to 90 degrees
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Connections:
- R1 pad 2: Net-(R1-Pad2) -> Net-(J1-Pad8)
- R2 pad 2: Net-(R2-Pad2) -> Net-(J1-Pad8)
- R3 pad 2: Net-(R3-Pad2) -> Net-(J1-Pad8)
- R4 pad 2: Net-(R4-Pad2) -> Net-(J1-Pad8)
- R5 pad 2: Net-(R5-Pad2) -> Net-(J1-Pad8)
- R6 pad 2: Net-(R6-Pad2) -> Net-(J1-Pad8)
- R7 pad 2: Net-(R7-Pad2) -> Net-(J1-Pad8)
Routing:
- net Net-(D16-Pad2): track 0.00 -> 529.7 mm
- net Net-(D15-Pad2): track 0.00 -> 502.1 mm
- net Net-(D14-Pad2): track 0.00 -> 455.1 mm
- net Net-(J2-Pad1): track 0.00 -> 441.3 mm
- net Net-(D13-Pad2): track 0.00 -> 436.1 mm, vias 0 -> 2
- net Net-(J2-Pad3): track 0.00 -> 422.0 mm, vias 0 -> 2
- net Net-(J2-Pad2): track 0.00 -> 421.1 mm
- net Net-(J2-Pad5): track 0.00 -> 386.9 mm, vias 0 -> 2
- net Net-(J2-Pad4): track 0.00 -> 383.5 mm
- net Net-(D12-Pad2): track 0.00 -> 383.2 mm
- net Net-(J2-Pad7): track 0.00 -> 361.8 mm, vias 0 -> 2
- net Net-(D11-Pad2): track 0.00 -> 359.3 mm, vias 0 -> 2
- net Net-(J2-Pad6): track 0.00 -> 346.3 mm
- net Net-(J1-Pad8): track 0.00 -> 328.1 mm, vias 0 -> 4
- net Net-(D10-Pad2): track 0.00 -> 309.8 mm
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Other:
- net class Default: clearance 0.254 -> 0.6; trace_width 0.254 -> 1.016
- rule trace_clearance: 0.254 -> 0.6
- rule trace_min: 0.254 -> 1.016

Commit message: edge novi .dxf
Other:
- board outline added: 259 x 313 mm
